Commit message: Initial status

File: resources/arm5e_gripper_bak.urdf (robot description, URDF)
Before this commit: robot arm5e_gripper, 3 links, 2 joints
Links:
- link part4_base: geometry visual mesh filename=package://UWSim/data/robot/ARM5E/ARM5E_part4_base.osg
- link part4_jaw1: geometry visual mesh filename=package://UWSim/data/robot/ARM5E/ARM5E_part4_jaw1long.osg
- link part4_jaw2: geometry visual mesh filename=package://UWSim/data/robot/ARM5E/ARM5E_part4_jaw2long.osg
